File: eagle/a78-simple-epi.brd (EAGLE design)
At the start: 50.2 x 49.8 mm, 35 parts, among them IC1 ATMEGA 328P, Q2 2N3904, Q3 2N3904

Commit message: patch
Routing:
- net +5V: track 93.5 -> 104.0 mm, vias 0 -> 2
Changed lines of the file:
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@@
 <plain>
 <wire x1="0" y1="60.6425" x2="0" y2="10.795" width="0" layer="20"/>
-<dimension x1="0" y1="9.8425" x2="50.165" y2="9.8425" x3="25.0825" y3="0" textsize="1.778" layer="20"/>
-<dimension x1="0" y1="60.96" x2="0" y2="10.795" x3="-5.08" y3="35.8775" textsize="1.778" layer="20"/>
 <wire x1="45.085" y1="10.795" x2="45.085" y2="27.94" width="0" layer="20"/>
 <wire x1="45.085" y1="27.94" x2="50.165" y2="27.94" width="0" layer="20"/>
@@
 <wire x1="50.165" y1="60.6425" x2="0" y2="60.6425" width="0" layer="20"/>
 <wire x1="0" y1="10.795" x2="45.085" y2="10.795" width="0" layer="20"/>
-<dimension x1="50.165" y1="60.96" x2="40.005" y2="60.96" x3="45.085" y3="63.8175" textsize="1.778" layer="20"/>
 <hole x="40.005" y="56.1975" drill="2.2"/>
-<dimension x1="50.4825" y1="55.5625" x2="50.4825" y2="60.6425" x3="53.34" y3="58.1025" textsize="1.778" layer="20"/>
 <text x="11.7475" y="16.51" size="2.54" layer="25">A78-SIMPLE EPI</text>
 <text x="12.3825" y="19.685" size="1.9304" layer="25">tdididit.com</text>
@@
 <contactref element="R10" pad="1"/>
 <contactref element="R11" pad="1"/>
-<wire x1="33.5525" y1="48.895" x2="37.5125" y2="48.895" width="0.4064" layer="1"/>
+<wire x1="33.5525" y1="48.895" x2="36.5125" y2="48.895" width="0.4064" layer="1"/>
+<wire x1="36.5125" y1="48.895" x2="37.5125" y2="48.895" width="0.4064" layer="1"/>
 <wire x1="37.5125" y1="48.895" x2="39.37" y2="50.7525" width="0.4064" layer="1"/>
 <wire x1="19.265" y1="41.275" x2="26.3525" y2="41.275" width="0.4064" layer="1"/>
@@
 <wire x1="26.7725" y1="39.6875" x2="26.7725" y2="38.6325" width="0.4064" layer="1"/>
 <wire x1="26.7725" y1="38.6325" x2="26.9875" y2="38.4175" width="0.4064" layer="1"/>
-<wire x1="26.9875" y1="38.4175" x2="37.2875" y2="38.4175" width="0.4064" layer="1"/>
+<wire x1="26.9875" y1="38.4175" x2="36.5125" y2="38.4175" width="0.4064" layer="1"/>
+<wire x1="36.5125" y1="38.4175" x2="37.1475" y2="38.4175" width="0.4064" layer="1"/>
+<wire x1="37.1475" y1="38.4175" x2="37.2875" y2="38.4175" width="0.4064" layer="1"/>
 <wire x1="37.2875" y1="38.4175" x2="38.565" y2="37.14" width="0.4064" layer="1"/>
 <wire x1="27.6225" y1="31.8525" x2="28.0425" y2="31.965" width="0.4064" layer="1"/>
@@
 <wire x1="9.8425" y1="57.785" x2="7.3025" y2="57.785" width="0.4064" layer="16"/>
 <wire x1="7.3025" y1="57.785" x2="6.0325" y2="59.055" width="0.4064" layer="16"/>
-<wire x1="37.2875" y1="38.4175" x2="37.5125" y2="48.895" width="0" layer="19" extent="1-1"/>
+<via x="36.5125" y="48.895" extent="1-16" drill="0.3302"/>
+<wire x1="36.5125" y1="48.895" x2="36.5125" y2="38.4175" width="0.4064" layer="16"/>
+<via x="36.5125" y="38.4175" extent="1-16" drill="0.3302"/>
 </signal>
 <signal name="N$14">

Commit message: update
Parts:
- added RST, TP1: TPB1,27, testpad:B1,27
Connections:
- net GND: now also TP1.TP
- net RST: now also RST.TP
Routing:
- net RST: track 50.2 -> 53.3 mm
Changed lines of the file:
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@@
 <attribute name="VALUE" x="3.302" y="53.721" size="1.27" layer="27" rot="R90"/>
+</element>
+<element name="TP1" library="testpad" package="B1,27" value="TPB1,27" x="1.5875" y="38.735" smashed="yes">
+<attribute name="TP_SIGNAL_NAME" value="" x="0.9525" y="36.83" size="1" layer="37"/>
+<attribute name="VALUE" x="0.9525" y="37.973" size="0.0254" layer="27"/>
+</element>
+<element name="RST" library="testpad" package="B1,27" value="TPB1,27" x="1.5875" y="41.275" smashed="yes">
+<attribute name="TP_SIGNAL_NAME" value="" x="0.9525" y="39.37" size="1" layer="37"/>
+<attribute name="NAME" x="2.8575" y="39.4335" size="0.8128" layer="25" ratio="10"/>
+<attribute name="VALUE" x="0.9525" y="40.513" size="0.0254" layer="27"/>
 </element>
 </elements>
@@
 <wire x1="41.275" y1="58.42" x2="41.5925" y2="58.42" width="0.24" layer="1"/>
 <wire x1="41.5925" y1="58.42" x2="41.91" y2="58.1025" width="0.24" layer="1"/>
+<contactref element="TP1" pad="TP"/>
 </signal>
 <signal name="LEFT">
@@
 <wire x1="19.05" y1="40.005" x2="4.1275" y2="40.005" width="0.4064" layer="1"/>
 <wire x1="4.1275" y1="40.005" x2="3.81" y2="40.3225" width="0.4064" layer="1"/>
-<wire x1="3.81" y1="40.3225" x2="3.81" y2="43.815" width="0.4064" layer="1"/>
 <contactref element="JP1" pad="5"/>
 <contactref element="C5" pad="1"/>
+<wire x1="3.81" y1="40.3225" x2="3.81" y2="43.815" width="0.4064" layer="1"/>
 <wire x1="1.27" y1="53.76" x2="1.3725" y2="53.76" width="0.4064" layer="1"/>
 <wire x1="3.2775" y1="53.76" x2="3.4925" y2="53.975" width="0.4064" layer="1"/>
 <wire x1="3.2775" y1="53.76" x2="1.3725" y2="53.76" width="0.4064" layer="1"/>
 <wire x1="1.3725" y1="53.76" x2="1.27" y2="53.6575" width="0.4064" layer="1"/>
-<wire x1="1.27" y1="53.6575" x2="1.27" y2="44.45" width="0.4064" layer="1"/>
-<wire x1="1.27" y1="44.45" x2="1.905" y2="43.815" width="0.4064" layer="1"/>
-<wire x1="1.905" y1="43.815" x2="3.9125" y2="43.815" width="0.4064" layer="1"/>
+<wire x1="1.27" y1="53.6575" x2="1.27" y2="43.815" width="0.4064" layer="1"/>
+<wire x1="1.27" y1="43.815" x2="3.9125" y2="43.815" width="0.4064" layer="1"/>
 <wire x1="19.9644" y1="37.8587" x2="19.9644" y2="31.3563" width="0.4064" layer="16"/>
+<contactref element="RST" pad="TP"/>
+<wire x1="1.5875" y1="41.275" x2="1.27" y2="41.5925" width="0.4064" layer="1"/>
+<wire x1="1.27" y1="41.5925" x2="1.27" y2="43.815" width="0.4064" layer="1"/>
 </signal>
 <signal name="MOSI">
