File: eagle/a78-simple-epi.sch (EAGLE design)
At the start: 35 parts, among them IC1 ATMEGA 328P, Q2 2N3904, Q3 2N3904

Commit message: update
Parts:
- added RST, TP1: TPB1,27, testpad:TPB1,27
Connections:
- net GND: now also TP1.TP
- net RST: now also RST.TP
Changed lines of the file:
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@@
 <part name="C5" library="resistor" deviceset="C-EU" device="C0603"/>
 <part name="FRAME1" library="frames" deviceset="DINA4_L" device=""/>
+<part name="TP1" library="testpad" deviceset="TP" device="B1,27"/>
+<part name="RST" library="testpad" deviceset="TP" device="B1,27"/>
+<part name="GND9" library="supply1" deviceset="GND" device=""/>
 </parts>
 <sheets>
@@
 <instance part="FRAME1" gate="G$1" x="0" y="0"/>
 <instance part="FRAME1" gate="G$2" x="162.56" y="0"/>
+<instance part="TP1" gate="G$1" x="12.7" y="111.76"/>
+<instance part="RST" gate="G$1" x="22.86" y="111.76"/>
+<instance part="GND9" gate="1" x="12.7" y="104.14"/>
 </instances>
 <busses>
@@
 <wire x1="142.24" y1="17.78" x2="142.24" y2="15.24" width="0.1524" layer="91"/>
 <pinref part="GND12" gate="1" pin="GND"/>
+</segment>
+<segment>
+<pinref part="TP1" gate="G$1" pin="TP"/>
+<pinref part="GND9" gate="1" pin="GND"/>
+<wire x1="12.7" y1="106.68" x2="12.7" y2="109.22" width="0.1524" layer="91"/>
 </segment>
 </net>
@@
 <label x="152.4" y="27.94" size="1.778" layer="95"/>
 </segment>
-</net>
+<segment>
+<pinref part="RST" gate="G$1" pin="TP"/>
+<wire x1="22.86" y1="109.22" x2="22.86" y2="106.68" width="0.1524" layer="91"/>
+<wire x1="22.86" y1="106.68" x2="33.02" y2="106.68" width="0.1524" layer="91"/>
+<label x="27.94" y="106.68" size="1.778" layer="95"/>
+</segment>
+</net>
